File: HDK/GD32F307_Mini_Board/GD32F307_Mini_Board.sch (KiCad schematic (older format))
At the start: 0 parts

Commit message: 增加 NAND ETH LCD 原理图
Other:
- note added: "E2PROM\n\n"
- note added: "Ethernet"
- note added: "GD32F307VCT6\n"
- note added: "LCD\n"
- note added: "Nand_Flash\n"
- note added: "Power\n\n"
- note added: "Spi_Flash\n\n"
- note added: "interface\n\n"
