File: HDK/GD32F307_Mini_Board/main.sch (KiCad schematic (older format))
At the start: 29 parts

Commit message: 增加 NAND ETH LCD 原理图
Parts:
- removed U?: STM32F303VCTx, Package_QFP:LQFP-100_14x14mm_P0.5mm, symbol MCU_ST_STM32F3:STM32F303VCTx
- added U?: STM32F107VCTx, Package_QFP:LQFP-100_14x14mm_P0.5mm, symbol MCU_ST_STM32F1:STM32F107VCTx
- C? (x2): Comment 10pF (100) 5% 50V -> 10pF
- J?: value Conn_02x10_Odd_Even -> JTAG
- Y?: Comment 32.768KHz ±20ppm 12.5pF -> 32.768KHz
Connections:
- net labels added: ADC_IN, BackLight, EXMC_A16, EXMC_A17, EXMC_A23, EXMC_D0, EXMC_D1, EXMC_D10, EXMC_D11, EXMC_D12, EXMC_D13, EXMC_D14, EXMC_D15, EXMC_D2, EXMC_D3, EXMC_D4, EXMC_D5, EXMC_D6, EXMC_D7, EXMC_D8, EXMC_D9, EXMC_NOE, EXMC_NWAIT, EXMC_NWE, I2C_SCL, I2C_SDA, LCD_CS, NAND_CS, RMII_CRS_DV, RMII_INT, RMII_MDC, RMII_MDIO, RMII_REF_CLK, RMII_RXD0, RMII_RXD1, RMII_TXD0, RMII_TXD1, RMII_TX_EN, SPI_CLK, SPI_CS, SPI_MISO, SPI_MOSI, T_CLK, T_CS, T_MISO, T_MOSI, T_PEN, UART0_RXD, UART0_TXD
- wire segments 116 -> 165
Other:
- moved on the sheet: C?, Y?
